File: source/Cheap FOCer 2 60mm.kicad_pcb (KiCad board)
At the start: 2 copper layers, 59.1 x 99.9 mm, 193 parts, among them J1 Conn_01x02, J2 Conn_01x07, J3 Conn_01x03, J4 On/Off, J5 UNUSED MCU PINS, J6 Conn_01x03, P1 MOTOR1, P2 MOTOR1, P3 MOTOR1, P4 HALL/Encoder, P5 SWD, Q1 NCEP60T20, Q2 NCEP60T20, Q3 NCEP60T20, Q4 NCEP60T20, Q5 NCEP60T20, Q6 NCEP60T20, U1 AMS1117-3.3, U2 DRV8301, U3 TP2604-SR, U4 TJA1051T/3/1J, U5 STM32F405RGT6, U6 BMI160, X1 8MHz 10ppm (X50328MSB2GI)

Commit message: bumped the project to kicad 10
Parts:
- C13: value 120p -> 150p
- D1, D2: value SMF05CT1G -> SMF05CT1G
Connections:
- U2 pad 12: Net-(U2-Pad12) -> unconnected-(U2-DC_CAL-Pad12)
- U2 pad 4: Net-(U2-Pad4) -> unconnected-(U2-PWRGD-Pad4)
- U2 pad 5: Net-(U2-Pad5) -> unconnected-(U2-OCTW-Pad5)
- U6 pad 10: Net-(U6-Pad10) -> unconnected-(U6-OCSB-Pad10)
- U6 pad 11: Net-(U6-Pad11) -> unconnected-(U6-OSDO-Pad11)
- U6 pad 2: Net-(U6-Pad2) -> unconnected-(U6-ASDX-Pad2)
- U6 pad 3: Net-(U6-Pad3) -> unconnected-(U6-ASCX-Pad3)
- U6 pad 4: Net-(U6-Pad4) -> unconnected-(U6-INT1-Pad4)
- U6 pad 9: Net-(U6-Pad9) -> unconnected-(U6-INT2-Pad9)
- USB1 pad 1: Net-(USB1-Pad1) -> unconnected-(USB1-VBUS-Pad1)
- USB1 pad 4: Net-(USB1-Pad4) -> unconnected-(USB1-ID-Pad4)
- USB1 pad 6: GND -> (no net)
Other:
- net class Default removed

Commit message: added gitignore
Connections:
- net /CAN bus transceiver/CANH renamed /Channel A/CAN bus transceiver/CANH
- net /CAN bus transceiver/CANL renamed /Channel A/CAN bus transceiver/CANL
- net /CAN bus transceiver/CAN_RX renamed /Channel A/CAN bus transceiver/CAN_RX
- net /CAN bus transceiver/CAN_TX renamed /Channel A/CAN bus transceiver/CAN_TX
- net /Filters/HALL1_IN renamed /Channel A/Filters/HALL1_IN
- net /Filters/HALL2_IN renamed /Channel A/Filters/HALL2_IN
- net /Filters/TEMP_IN renamed /Channel A/Filters/TEMP_IN
- net /HALL3 renamed /Channel A/HALL3
- net /MCU/ADC_TEMP renamed /Channel A/MCU/ADC_TEMP
- net /MCU/AN_IN renamed /Channel A/MCU/AN_IN
- net /MCU/BR_SO1 renamed /Channel A/MCU/BR_SO1
- net /MCU/BR_SO2 renamed /Channel A/MCU/BR_SO2
- net /MCU/BR_SO3 renamed /Channel A/MCU/BR_SO3
- net /MCU/CS renamed /Channel A/MCU/CS
- net /MCU/EN_GATE renamed /Channel A/MCU/EN_GATE
- net /MCU/FAULT renamed /Channel A/MCU/FAULT
- net /MCU/H1 renamed /Channel A/MCU/H1
- net /MCU/H2 renamed /Channel A/MCU/H2
- net /MCU/H3 renamed /Channel A/MCU/H3
- net /MCU/L1 renamed /Channel A/MCU/L1
- net /MCU/L2 renamed /Channel A/MCU/L2
- net /MCU/L3 renamed /Channel A/MCU/L3
- net /MCU/LED_GREEN renamed /Channel A/MCU/LED_GREEN
- net /MCU/LED_RED renamed /Channel A/MCU/LED_RED
- net /MCU/MISO_ADC_EXT2 renamed /Channel A/MCU/MISO_ADC_EXT2
- net /MCU/RX_SDA_NSS renamed /Channel A/MCU/RX_SDA_NSS
- net /MCU/SCK_ADC_EXT renamed /Channel A/MCU/SCK_ADC_EXT
- net /MCU/SDI renamed /Channel A/MCU/SDI
- net /MCU/SDO renamed /Channel A/MCU/SDO
- net /MCU/SENS1 renamed /Channel A/MCU/SENS1
- net /MCU/SENS2 renamed /Channel A/MCU/SENS2
- net /MCU/SENS3 renamed /Channel A/MCU/SENS3
- net /MCU/SERVO renamed /Channel A/MCU/SERVO
- net /MCU/SLCK renamed /Channel A/MCU/SLCK
- net /MCU/TX_SCL_MOSI renamed /Channel A/MCU/TX_SCL_MOSI
- net /MCU/USB_DM renamed /Channel A/MCU/USB_DM
- net /MCU/USB_DP renamed /Channel A/MCU/USB_DP
- net /MISO_RX_SCL_IN renamed /Channel A/MISO_RX_SCL_IN
- net /Mosfet driver/GH_A renamed /Channel A/Mosfet driver/GH_A
- net /Mosfet driver/GH_B renamed /Channel A/Mosfet driver/GH_B
- net /Mosfet driver/GH_C renamed /Channel A/Mosfet driver/GH_C
- net /Mosfet driver/GL_A renamed /Channel A/Mosfet driver/GL_A
- net /Mosfet driver/GL_B renamed /Channel A/Mosfet driver/GL_B
- net /Mosfet driver/GL_C renamed /Channel A/Mosfet driver/GL_C
- net /Mosfet driver/H1_LOW renamed /Channel A/Mosfet driver/H1_LOW
- net /Mosfet driver/H1_VS renamed /Channel A/Mosfet driver/H1_VS
- net /Mosfet driver/H2_LOW renamed /Channel A/Mosfet driver/H2_LOW
- net /Mosfet driver/H2_VS renamed /Channel A/Mosfet driver/H2_VS
- net /Mosfet driver/H3_LOW renamed /Channel A/Mosfet driver/H3_LOW
- net /Mosfet driver/H3_VS renamed /Channel A/Mosfet driver/H3_VS
- net /RX_SDA_IN renamed /Channel A/RX_SDA_IN
- net /SCK_ADC_EXT_IN renamed /Channel A/SCK_ADC_EXT_IN
- net /TX_SCL_MOSI_IN renamed /Channel A/TX_SCL_MOSI_IN
