File: source/Cheap FOCer 2 60mm.kicad_sch (KiCad schematic)
At the start: 49 parts, among them J1 Conn_01x02, J2 Conn_01x07, J3 Conn_01x03, J6 Conn_01x03, P1 MOTOR1, P2 MOTOR1, P3 MOTOR1, P4 HALL/Encoder

Commit message: another fix for version bump
Parts:
- removed C1: 100n, Capacitor_SMD:C_0603_1608Metric, symbol BLDC_4-rescue:C-RESCUE-BLDC_4
- removed C2, C3: 0.01uF, Capacitor_SMD:C_0603_1608Metric, symbol BLDC_4-rescue:C-RESCUE-BLDC_4
- removed C4: .01uF, Capacitor_SMD:C_0603_1608Metric, symbol BLDC_4-rescue:C-RESCUE-BLDC_4
- removed D1, D2: SMF05CT1G, Package_TO_SOT_SMD:SOT-363_SC-70-6, symbol Power_Protection:SP0505BAHT
- removed D3: RED, LED_SMD:LED_0603_1608Metric, symbol Device:LED
- removed D4: GRN, LED_SMD:LED_0603_1608Metric, symbol Device:LED
- removed D5: BLU, LED_SMD:LED_0603_1608Metric, symbol Device:LED
- removed F1, F2, F3: Fiducial, Fiducial:Fiducial_1mm_Dia_2mm_Outer, symbol Mechanical:Fiducial
- removed H1, H13, H2, H5, H6, H8: MountingHole, MountingHole:MountingHole_3.2mm_M3_ISO14580_Pad, symbol Mechanical:MountingHole
- removed H3: SLJ, shapes3D:Sam_J, symbol Mechanical:MountingHole
- removed H4: Open Hardware Logo, Symbol:OSHW-Logo2_9.8x8mm_SilkScreen, symbol Mechanical:MountingHole
- removed H7: MountingHole, MountingHole:MountingHole_3.2mm_M3_ISO14580_Pad, symbol Mechanical:MountingHole_Pad
- removed H9: KiCAD Logo, Symbol:KiCad-Logo2_5mm_SilkScreen, symbol Mechanical:MountingHole
- removed J1: Conn_01x02, Connector_JST:JST_PH_B2B-PH-K_1x02_P2.00mm_Vertical, symbol Connector_Generic:Conn_01x02
- removed J2: Conn_01x07, Connector_JST:JST_PH_B7B-PH-K_1x07_P2.00mm_Vertical, symbol Connector_Generic:Conn_01x07
- removed J3: Conn_01x03, Connector_JST:JST_PH_B3B-PH-K_1x03_P2.00mm_Vertical, symbol Connector_Generic:Conn_01x03
- removed J6: Conn_01x03, Connector_PinHeader_2.54mm:PinHeader_1x02_P2.54mm_Vertical, symbol Connector_Generic:Conn_01x02
- removed NEG3: MOTOR3, CRF1:1pin_4mm, symbol BLDC_4-rescue:CONN_1
- removed P1, P2, P3: MOTOR1, CRF1:1pin_4mm, symbol BLDC_4-rescue:CONN_1
- removed P4: HALL/Encoder, Connector_JST:JST_PH_B6B-PH-K_1x06_P2.00mm_Vertical, symbol Connector_Generic:Conn_01x06
- removed POS1: POS, CRF1:1pin_4mm, symbol BLDC_4-rescue:CONN_1
- removed R1: 39k, Resistor_SMD:R_0603_1608Metric, symbol BLDC_4-rescue:R-RESCUE-BLDC_4
- removed R10, R11, R5, R6, R7, R8, R9: 100R, Resistor_SMD:R_0603_1608Metric, symbol BLDC_4-rescue:R-RESCUE-BLDC_4
- removed R12, R2: 2k2, Resistor_SMD:R_0603_1608Metric, symbol BLDC_4-rescue:R-RESCUE-BLDC_4
- removed R3, R4: 22R, Resistor_SMD:R_0603_1608Metric, symbol BLDC_4-rescue:R-RESCUE-BLDC_4
- removed R40, R68, R71, R72: DNP, Resistor_SMD:R_0603_1608Metric, symbol BLDC_4-rescue:R-RESCUE-BLDC_4
- removed USB1: USB Micro U-D-M5DD-W-1, Connector_USB:USB_Micro-B_Wuerth_614105150721_Vertical, symbol Connector:USB_B_Micro
Connections:
- no-connect marks 2 -> 0
Other:
- removed sheet CAN bus transceiver
- removed sheet Filters
- removed sheet IMU
- removed sheet MCU
- removed sheet Mosfet driver
- removed sheet NTC temp sensor
- removed sheet Power MOSFETS
- added sheet Channel A (CH-A.kicad_sch)
- added sheet Channel B (CH-B.kicad_sch)
- note added: "Cheap F Cer 2 - 2 channels"
- note removed: "Cheap F Cer 2"
- note removed: "Connect signal ground and power ground in one place only"
- note removed: "Fiducials"
- note removed: "Logos"
- note removed: "Mounting Holes"
- note removed: "Pads for auxillary 5V out"
- note removed: "Power Pads"
- note removed: "Pull up and Pull down resistors on ADC channels. DNP by default. Use 10k resistors if needed"
- note removed: "Voltage supply (0 - 51v)"
